File: src/esp32c3/hardware/noisemeter.kicad_pcb (KiCad board)
At the start: 2 copper layers, 50 x 50 mm, 32 parts, among them J1 USB_B_Micro, J2 Conn_01x04_Pin, SW1 SW_Push, U1 AP2112K-3.3, U2 ESP32-C3-MINI-1-N4

Commit message: move bringup to esp32c3 folder
Other:
- board text added: "FILES: DRL=DRILL TOOL SIZE INFORMATION (MM) GM1=OUTLINE GTL=TOP LAYER GBL=BOT LAYER GTO=SILKSCREEN TOP GBO=SILKSCREEN BOT GTS=SOLDER MASK TOP GBS=SOLDER MASK BOT GTP=TOP STENCIL GBP=BOTTOM STENCIL POS=TOP PLACE FILE BOM=BILL OF MATERIALS SCHEMATIC FABDRAWING"
- board text added: "NOTES 1. PRINTED CIRCUIT BOARD MADE FROM NEMA GRADE FR-4 EPOXY LAMINATE. 2. ALL DIMENSIONS ARE GIVEN IN MILLIMETERS. 3. CIRCUIT PATHS ARE FOR REFERENCE ONLY. 4. HOLE SIZES SHOWN ARE FINISHED DIAMETERS AFTER PLATING. 5. APPLY GREEN SOLDER MASK ON PLATED SURFACES. 6. SILKSCREEN TOP AND BOTTOM SIDES USING WHITE INK. 7. ALL VIAS ARE TENTED ON BOTH SIDES. 8. 2 COPPER LAYERS. 9. 1.6MM BOARD THICKNESS. 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"
Changed lines of the file:
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@@
   (title_block
     (title "Noisemeter Device")
-    (date "2024-01-10")
+    (date "2024-01-22")
     (company "Civic Tech Toronto")
     (comment 1 "Drawn by Clyne Sullivan")
@@
       (plot_on_all_layers_selection 0x0000000_00000000)
       (disableapertmacros false)
-      (usegerberextensions false)
+      (usegerberextensions true)
       (usegerberattributes true)
       (usegerberadvancedattributes true)
@@
       (outputformat 1)
       (mirror false)
-      (drillshape 1)
+      (drillshape 0)
       (scaleselection 1)
-      (outputdirectory "")
+      (outputdirectory "production/20240121_081307/")
     )
   )
@@
     (effects (font (size 1 1) (thickness 0.15)) (justify right))
   )
+  (gr_text "FILES:\n\nDRL=DRILL TOOL SIZE INFORMATION (MM)\nGM1=OUTLINE\nGTL=TOP LAYER\nGBL=BOT LAYER\nGTO=SILKSCREEN TOP\nGBO=SILKSCREEN BOT\nGTS=SOLDER MASK TOP\nGBS=SOLDER MASK BOT\nGTP=TOP STENCIL\nGBP=BOTTOM STENCIL\nPOS=TOP PLACE FILE\nBOM=BILL OF MATERIALS\nSCHEMATIC\nFABDRAWING" (at 219.5 121) (layer "F.SilkS")
+    (effects (font (size 1.5 1.5) (thickness 0.15)) (justify left top))
+  )
+  (gr_text "NOTES\n\n 1. PRINTED CIRCUIT BOARD MADE FROM NEMA GRADE FR-4 EPOXY LAMINATE.\n 2. ALL DIMENSIONS ARE GIVEN IN MILLIMETERS.\n 3. CIRCUIT PATHS ARE FOR REFERENCE ONLY.\n 4. HOLE SIZES SHOWN ARE FINISHED DIAMETERS AFTER PLATING.\n 5. APPLY GREEN SOLDER MASK ON PLATED SURFACES.\n 6. SILKSCREEN TOP AND BOTTOM SIDES USING WHITE INK.\n 7. ALL VIAS ARE TENTED ON BOTH SIDES.\n 8. 2 COPPER LAYERS.\n 9. 1.6MM BOARD THICKNESS.\n10. COPPER THICKNESS 1 OZ.\n11. LEAD-FREE HASL SURFACE FINISH." (at 38.75 139) (layer "F.SilkS")
+    (effects (font (size 1.5 1.5) (thickness 0.15)) (justify left top))
+  )
   (gr_text "VCC" (at 167 85.5 90) (layer "F.SilkS")

Commit message: schematic/layout draft
Parts:
- removed D2: LED, LED_SMD:LED_0603_1608Metric
- removed J2: Conn_01x04_Pin, Connector_PinHeader_2.54mm:PinHeader_1x05_P2.54mm_Vertical
- removed R1, R7: 0, Resistor_SMD:R_0603_1608Metric
- removed R9: 150, Resistor_SMD:R_0603_1608Metric
- removed TP2, TP3: TestPoint, TestPoint:TestPoint_Pad_D1.5mm
- R8: value 150 -> 51
- SW1: footprint Button_Switch_SMD:SW_SPST_TL3305A -> Button_Switch_SMD:SW_SPST_EVQP7A
- moved D1 36.1 mm to (143.0, 124.0)
- moved SW1 24.6 mm to (138.0, 123.2), turned to 0 degrees
- moved TP1 24.2 mm to (155.8, 93.5), turned to 0 degrees
- moved R8 15.8 mm to (145.0, 94.0), turned to -90 degrees
- moved C2 7.48 mm to (146.8, 114.0), turned to 0 degrees
- moved C6 1.99 mm to (164.8, 96.8), turned to 90 degrees
- moved R4 1.82 mm to (141.2, 87.5)
- moved C4 1.68 mm to (141.2, 82.5), turned to 90 degrees
- moved R6 1.45 mm to (153.2, 94.0), turned to -90 degrees
- moved C5 1.35 mm to (139.5, 82.8), turned to 90 degrees
- moved C1 1.03 mm to (142.0, 89.8)
- moved C3 1.02 mm to (139.5, 113.8), turned to -90 degrees
- moved R2 1.00 mm to (149.2, 94.0)
- moved R3 1.00 mm to (150.8, 94.0)
- moved C7 0.62 mm to (166.2, 96.8), turned to 90 degrees
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Connections:
- net BUTTON renamed FACT_RESET
- net LED1 renamed STAT_LED
- MK1 pad 2: Net-(MK1-SELECT) -> GND
- TP1 pad 1: VBUS -> Net-(U2-IO9)
- U2 pad 16: Net-(U2-IO10) -> unconnected-(U2-IO10-Pad16)
- U2 pad 21: Net-(U2-IO7) -> unconnected-(U2-IO7-Pad21)
- U2 pad 23: BOOT -> Net-(U2-IO9)
- U2 pad 30: /RX -> unconnected-(U2-RXD0-Pad30)
- U2 pad 31: /TX -> unconnected-(U2-TXD0-Pad31)
- U2 pad 6: LED2 -> unconnected-(U2-IO3-Pad6)
Routing:
- net Net-(D1-K): track 1.64 -> 40.9 mm, vias 0 -> 2
- net +3V3: track 15.5 -> 53.8 mm, vias 4 -> 5
- net BOOT: track 25.3 -> 0.00 mm, vias 2 -> 0
- net MIC_WS: track 23.7 -> 45.8 mm
- net MIC_BCLK: track 21.3 -> 43.1 mm
- net MIC_DATA_OUT: track 21.9 -> 41.2 mm
- net FACT_RESET: track 25.8 -> 44.8 mm
- net LED2: track 15.6 -> 0.00 mm, vias 2 -> 0
- net STAT_LED: track 17.7 -> 2.11 mm, vias 2 -> 0
- net /RX: track 9.64 -> 0.00 mm
- net /TX: track 7.55 -> 0.00 mm
- net Net-(U2-IO10): track 7.33 -> 0.00 mm
- net Net-(J2-Pin_2): track 7.19 -> 0.00 mm
- net Net-(U2-IO7): track 6.12 -> 0.00 mm
- net Net-(U2-IO9): track 0.00 -> 3.07 mm
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- removed copper zone on B.Cu, net +3V3
Other:
- board text added: "rev2"
- board text removed: "BOOT"
- board text removed: "GND"
- board text removed: "RX"
- board text removed: "Reset"
- board text removed: "TX"
- board text removed: "VCC"

Commit message: redesign for 1551SFL case
Parts:
- removed H3, H4: MountingHole_Pad, MountingHole:MountingHole_2.5mm
- moved H2 41.5 mm to (171.5, 79.5)
- moved SW1 40.8 mm to (171.7, 100.2), turned to 90 degrees
- moved J1 37.0 mm to (171.2, 92.0), turned to 90 degrees
- moved MK1 36.6 mm to (134.2, 92.0), turned to -90 degrees
- moved D1 35.2 mm to (172.5, 104.7), turned to -90 degrees
- moved C3 28.5 mm to (165.0, 101.0), turned to 0 degrees
- moved C7 28.1 mm to (138.2, 94.2), turned to -90 degrees
- moved R10 27.9 mm to (139.0, 92.0), turned to 0 degrees
- moved C2 27.5 mm to (164.5, 93.0), turned to 90 degrees
- moved C6 25.1 mm to (139.8, 94.2), turned to -90 degrees
- moved U1 25.0 mm to (163.5, 97.7), turned to -90 degrees
- moved H1 17.0 mm to (133.0, 104.5)
- moved U2 9.73 mm to (158.8, 79.3)
- moved R3 9.70 mm to (159.5, 89.8)
- moved R2 9.47 mm to (157.8, 89.8)
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Routing:
- net USB_D_P: track 41.2 -> 11.7 mm
- net USB_D_N: track 40.3 -> 11.7 mm
- net MIC_WS: track 45.8 -> 21.7 mm, vias 2 -> 0
- net FACT_RESET: track 44.8 -> 65.3 mm
- net Net-(D1-K): track 40.9 -> 61.0 mm
- net MIC_DATA_OUT: track 41.2 -> 24.6 mm, vias 2 -> 0
- net MIC_BCLK: track 43.1 -> 26.9 mm, vias 2 -> 0
- net +3V3: track 53.8 -> 49.4 mm, vias 5 -> 3
- net VBUS: track 3.32 -> 4.10 mm
- net Net-(U2-EN): track 3.68 -> 4.43 mm
- net IO2: track 2.25 -> 3.00 mm
- net GND: vias 8 -> 23
- added copper zone on B.Cu, net +3V3
Other:
- board size 50 x 50 mm -> 44 x 37.8 mm
- board text added: ";.x_t} {\H0.62500x;(Part number and text placement/orientation on our products are }{\H0.62500x;subject to change,} {\H0.62500x;we do not recommend using them as a locating reference for }{\H0.62500x;modification purposes)}"
- board text added: "A"
- board text added: "B"
- board text added: "END VIEW"
- board text added: "INSIDE BOX"
- board text added: "INSIDE LID"
- board text added: "MAXIMUM"
- board text added: "P.C. BOARD SIZE"
- board text added: "SECTION A-A"
- board text added: "SECTION B-B"
- board text added: "SIDE VIEW"
- board text added: "TOP VIEW"
- board text added: "locked"
- board text added: "{\H2.0000;Dimensions:}\fArial|b0|i0;{\H2.0000; mm [inches]}"
- board text added: "{\H2.0000;www.hammondmfg.com}"
- board text removed: "Mic port"
