File: src/esp32c3/hardware/noisemeter.kicad_sch (KiCad schematic)
At the start: 32 parts, among them J1 USB_B_Micro, J2 Conn_01x04_Pin, SW1 SW_Push, U1 AP2112K-3.3, U2 ESP32-C3-MINI-1-N4

Commit message: schematic/layout draft
Parts:
- removed D2: LED, LED_SMD:LED_0603_1608Metric, symbol Device:LED
- removed J2: Conn_01x04_Pin, Connector_PinHeader_2.54mm:PinHeader_1x05_P2.54mm_Vertical, symbol Connector:Conn_01x05_Pin
- removed R1, R7: 0, Resistor_SMD:R_0603_1608Metric, symbol Device:R_US
- removed R9: 150, Resistor_SMD:R_0603_1608Metric, symbol Device:R_US
- removed TP1, TP3: TestPoint, TestPoint:TestPoint_Pad_D1.5mm, symbol Connector:TestPoint
- R8: value 150 -> 51; Part Number RC0603JR-07150RL -> RC0603JR-0751RL
- SW1: footprint Button_Switch_SMD:SW_SPST_TL3305A -> Button_Switch_SMD:SW_SPST_EVQP7A; Part Number TL3305AF260QG -> EVQ-P7A01P
- renumbered TP2 to TP1
Connections:
- net GND: now also MK1.2 (SELECT)
- net at U2.21 (IO7): no longer TP1.1
- net BOOT: no longer names the net of U2.23 (IO9)
- net BOOT: now also TP1.1
- net BUTTON renamed FACT_RESET
- net LED1 renamed STAT_LED
- net LED2: no longer names the net of U2.6 (IO3)
- net RX: no longer names the net of U2.30 (RXD0)
- net TX: no longer names the net of U2.31 (TXD0)
- no-connect marks 1 -> 6
Other:
- note added: "Status/diagnostic indicator"
- note removed: "Programming connector: Use any USB/serial adapter. Enter bootloader by bridging BOOT to GND during power-on or reset."
- note removed: "Status/diagnostic LED indicators"
- moved on the sheet: C1, R2, R3, R4, R8, TP1

Commit message: redesign for 1551SFL case
Parts:
- removed H3, H4: MountingHole_Pad, MountingHole:MountingHole_2.5mm, symbol Mechanical:MountingHole
Other:
- moved on the sheet: H1, H2
Changed lines of the file:
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@@
     )
   )
-  (symbol (lib_id "Mechanical:MountingHole") (at 145.415 176.53 0) (unit 1)
-    (in_bom yes) (on_board yes) (dnp no) (fields_autoplaced)
-    (property "Reference" "H2" (at 147.955 173.99 0)
+  (symbol (lib_id "Mechanical:MountingHole") (at 139.7 184.15 0) (unit 1)
+    (in_bom yes) (on_board yes) (dnp no) (fields_autoplaced)
+    (property "Reference" "H2" (at 142.24 181.61 0)
       (effects (font (size 1.27 1.27)) (justify left))
     )
-    (property "Value" "MountingHole_Pad" (at 147.955 176.53 0)
+    (property "Value" "MountingHole_Pad" (at 142.24 184.15 0)
       (effects (font (size 1.27 1.27)) (justify left))
     )
-    (property "Footprint" "MountingHole:MountingHole_2.5mm" (at 145.415 176.53 0)
-      (effects (font (size 1.27 1.27)) hide)
-    )
-    (property "Datasheet" "~" (at 145.415 176.53 0)
+    (property "Footprint" "MountingHole:MountingHole_2.5mm" (at 139.7 184.15 0)
+      (effects (font (size 1.27 1.27)) hide)
+    )
+    (property "Datasheet" "~" (at 139.7 184.15 0)
       (effects (font (size 1.27 1.27)) hide)
     )
@@
     )
   )
-  (symbol (lib_id "Mechanical:MountingHole") (at 145.415 189.23 0) (unit 1)
-    (in_bom yes) (on_board yes) (dnp no) (fields_autoplaced)
-    (property "Reference" "H4" (at 147.955 186.69 0)
-      (effects (font (size 1.27 1.27)) (justify left))
-    )
-    (property "Value" "MountingHole_Pad" (at 147.955 189.23 0)
-      (effects (font (size 1.27 1.27)) (justify left))
-    )
-    (property "Footprint" "MountingHole:MountingHole_2.5mm" (at 145.415 189.23 0)
-      (effects (font (size 1.27 1.27)) hide)
-    )
-    (property "Datasheet" "~" (at 145.415 189.23 0)
-      (effects (font (size 1.27 1.27)) hide)
-    )
-    (instances
-      (project "noisemeter"
-        (path "/2019f223-1307-408a-bf87-dad398f72c59"
-          (reference "H4") (unit 1)
-        )
-      )
-    )
-  )
   (symbol (lib_id "Device:R_US") (at 240.665 55.88 90) (unit 1)
     (in_bom yes) (on_board yes) (dnp no) (fields_autoplaced)
@@
     )
   )
-  (symbol (lib_id "Mechanical:MountingHole") (at 145.415 170.18 0) (unit 1)
-    (in_bom yes) (on_board yes) (dnp no) (fields_autoplaced)
-    (property "Reference" "H1" (at 147.955 167.64 0)
+  (symbol (lib_id "Mechanical:MountingHole") (at 139.7 177.8 0) (unit 1)
+    (in_bom yes) (on_board yes) (dnp no) (fields_autoplaced)
+    (property "Reference" "H1" (at 142.24 175.26 0)
       (effects (font (size 1.27 1.27)) (justify left))
     )
-    (property "Value" "MountingHole_Pad" (at 147.955 170.18 0)
+    (property "Value" "MountingHole_Pad" (at 142.24 177.8 0)
       (effects (font (size 1.27 1.27)) (justify left))
     )
-    (property "Footprint" "MountingHole:MountingHole_2.5mm" (at 145.415 170.18 0)
-      (effects (font (size 1.27 1.27)) hide)
-    )
-    (property "Datasheet" "~" (at 145.415 170.18 0)
+    (property "Footprint" "MountingHole:MountingHole_2.5mm" (at 139.7 177.8 0)
+      (effects (font (size 1.27 1.27)) hide)
+    )
+    (property "Datasheet" "~" (at 139.7 177.8 0)
       (effects (font (size 1.27 1.27)) hide)
     )
@@
         )
       )
-    )
-  )
-  (symbol (lib_id "Mechanical:MountingHole") (at 145.415 182.88 0) (unit 1)
-    (in_bom yes) (on_board yes) (dnp no) (fields_autoplaced)
-    (property "Reference" "H3" (at 147.955 180.34 0)
-      (effects (font (size 1.27 1.27)) (justify left))
-    )
-    (property "Value" "MountingHole_Pad" (at 147.955 182.88 0)
-      (effects (font (size 1.27 1.27)) (justify left))
-    )
-    (property "Footprint" "MountingHole:MountingHole_2.5mm" (at 145.415 182.88 0)
-      (effects (font (size 1.27 1.27)) hide)
-    )
-    (property "Datasheet" "~" (at 145.415 182.88 0)
-      (effects (font (size 1.27 1.27)) hide)
-    )
-    (instances
-      (project "noisemeter"
-        (path "/2019f223-1307-408a-bf87-dad398f72c59"
-          (reference "H3") (unit 1)
-        )
-      )
