File: hardware/pcb-rev1/noisemeter.kicad_pcb (KiCad board)
At the start: 2 copper layers, 44 x 37.8 mm, 23 parts, among them J1 USB_B_Micro, SW1 SW_Push, U1 AP2112K-3.3, U2 ESP32-C3-MINI-1-N4

Commit message: restore pcb-rev1 hw files
Parts:
- added D2: LED, LED_SMD:LED_0603_1608Metric, F.Cu at (133.2, 87.2)
- added H3: MountingHole_Pad, MountingHole:MountingHole_2.5mm, F.Cu at (171.0, 79.0)
- added H4: MountingHole_Pad, MountingHole:MountingHole_2.5mm, F.Cu at (129.0, 79.0)
- added J2: Conn_01x04_Pin, Connector_PinHeader_2.54mm:PinHeader_1x05_P2.54mm_Vertical, F.Cu at (169.6, 83.8)
- added R1: 0, Resistor_SMD:R_0603_1608Metric, F.Cu at (167.0, 91.8)
- added R7: 0, Resistor_SMD:R_0603_1608Metric, F.Cu at (167.0, 102.5)
- added R9: 150, Resistor_SMD:R_0603_1608Metric, F.Cu at (130.0, 87.2)
- added TP2: TestPoint, TestPoint:TestPoint_Pad_D1.5mm, F.Cu at (154.2, 96.5)
- added TP3: TestPoint, TestPoint:TestPoint_Pad_D1.5mm, F.Cu at (147.2, 98.0)
- R8: value 51 -> 150
- SW1: footprint Button_Switch_SMD:SW_SPST_EVQP7A -> Button_Switch_SMD:SW_SPST_TL3305A
- moved D1 42.2 mm to (133.2, 89.2), turned to 0 degrees
- moved SW1 41.7 mm to (130.0, 100.0), turned to -90 degrees
- moved H2 41.5 mm to (171.0, 121.0)
- moved J1 37.0 mm to (150.0, 122.2), turned to 0 degrees
- moved MK1 36.6 mm to (170.0, 100.0), turned to 90 degrees
- moved C2 33.2 mm to (139.3, 114.6), turned to 180 degrees
- moved TP1 31.6 mm to (145.2, 115.2), turned to 180 degrees
- moved C3 28.3 mm to (139.3, 112.8), turned to 180 degrees
- moved R10 27.9 mm to (165.7, 100.0), turned to 180 degrees
- moved C7 27.6 mm to (165.7, 97.0), turned to 180 degrees
- moved C6 26.3 mm to (165.7, 98.5), turned to 180 degrees
- moved U1 25.0 mm to (143.0, 112.0), turned to 180 degrees
- moved R8 22.8 mm to (130.0, 89.2), turned to 0 degrees
- moved H1 17.0 mm to (129.0, 121.0)
- moved R4 10.8 mm to (139.5, 88.0)
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Connections:
- net FACT_RESET renamed BUTTON
- net STAT_LED renamed LED1
- MK1 pad 2: GND -> Net-(MK1-SELECT)
- TP1 pad 1: Net-(U2-IO9) -> VBUS
- U2 pad 16: unconnected-(U2-IO10-Pad16) -> Net-(U2-IO10)
- U2 pad 21: unconnected-(U2-IO7-Pad21) -> Net-(U2-IO7)
- U2 pad 23: Net-(U2-IO9) -> BOOT
- U2 pad 30: unconnected-(U2-RXD0-Pad30) -> /RX
- U2 pad 31: unconnected-(U2-TXD0-Pad31) -> /TX
- U2 pad 6: unconnected-(U2-IO3-Pad6) -> LED2
Routing:
- net Net-(D1-K): track 61.0 -> 1.64 mm, vias 2 -> 0
- net BUTTON: track 65.3 -> 25.8 mm
- net +3V3: track 49.4 -> 15.5 mm, vias 3 -> 4
- net USB_D_P: track 11.7 -> 41.5 mm
- net USB_D_N: track 11.7 -> 40.7 mm
- net BOOT: track 0.00 -> 25.3 mm, vias 0 -> 2
- net LED2: track 0.00 -> 15.6 mm, vias 0 -> 2
- net LED1: track 2.26 -> 17.7 mm, vias 0 -> 2
- net /RX: track 0.00 -> 9.64 mm
- net /TX: track 0.00 -> 7.55 mm
- net Net-(U2-IO10): track 0.00 -> 7.33 mm
- net Net-(J2-Pin_2): track 0.00 -> 7.19 mm
- net Net-(U2-IO7): track 0.00 -> 6.12 mm
- net MIC_BCLK: track 26.9 -> 21.3 mm, vias 0 -> 2
- net Net-(U2-IO9): track 2.91 -> 0.00 mm
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Other:
- board size 44 x 37.8 mm -> 50 x 50 mm
- board text added: "BOOT"
- board text added: "GND"
- board text added: "Mic port"
- board text added: "RX"
- board text added: "Reset"
- board text added: "TX"
- board text added: "VCC"
- board text removed: ";.x_t} {\H0.62500x;(Part number and text placement/orientation on our products are }{\H0.62500x;subject to change,} {\H0.62500x;we do not recommend using them as a locating reference for }{\H0.62500x;modification purposes)}"
- board text removed: "A"
- board text removed: "B"
- board text removed: "END VIEW"
- board text removed: "INSIDE BOX"
- board text removed: "INSIDE LID"
- board text removed: "MAXIMUM"
- board text removed: "P.C. BOARD SIZE"
- board text removed: "SECTION A-A"
- board text removed: "SECTION B-B"
- board text removed: "SIDE VIEW"
- board text removed: "TOP VIEW"
- board text removed: "locked"
- board text removed: "rev2"
- board text removed: "{\H2.0000;Dimensions:}\fArial|b0|i0;{\H2.0000; mm [inches]}"
- board text removed: "{\H2.0000;www.hammondmfg.com}"
