File: hardware/pcb-rev1/noisemeter.kicad_sch (KiCad schematic)
At the start: 23 parts, among them J1 USB_B_Micro, SW1 SW_Push, U1 AP2112K-3.3, U2 ESP32-C3-MINI-1-N4

Commit message: restore pcb-rev1 hw files
Parts:
- added D2: LED, LED_SMD:LED_0603_1608Metric, symbol Device:LED
- added H3, H4: MountingHole_Pad, MountingHole:MountingHole_2.5mm, symbol Mechanical:MountingHole
- added J2: Conn_01x04_Pin, Connector_PinHeader_2.54mm:PinHeader_1x05_P2.54mm_Vertical, symbol Connector:Conn_01x05_Pin
- added R1, R7: 0, Resistor_SMD:R_0603_1608Metric, symbol Device:R_US
- added R9: 150, Resistor_SMD:R_0603_1608Metric, symbol Device:R_US
- added TP1, TP3: TestPoint, TestPoint:TestPoint_Pad_D1.5mm, symbol Connector:TestPoint
- R8: value 51 -> 150; Part Number RC0603JR-0751RL -> RC0603JR-07150RL
- SW1: footprint Button_Switch_SMD:SW_SPST_EVQP7A -> Button_Switch_SMD:SW_SPST_TL3305A; Part Number EVQ-P7A01P -> TL3305AF260QG
- renumbered TP1 to TP2
Connections:
- net +3V3: now also D2.2 (A), R1.2
- net GND: now also J2.5 (Pin_5), R7.1; no longer MK1.2 (SELECT)
- net VBUS: now also TP1.1
- net at U2.16 (IO10): now also TP3.1
- net at U2.21 (IO7): now also TP2.1
- net BOOT: now reaches U2.23 (IO9)
- net BOOT: now also J2.1 (Pin_1); no longer TP2.1
- net RX: now reaches U2.30 (RXD0)
- net RX: now also J2.3 (Pin_3)
- net TX: now reaches U2.31 (TXD0)
- net TX: now also J2.4 (Pin_4)
- net LED2: now reaches U2.6 (IO3)
- net LED2: now also R9.1
- net FACT_RESET renamed BUTTON
- net STAT_LED renamed LED1
- new net: D2.1 (K), R9.2
- new net: MK1.2 (SELECT), R7.2
- new net: J2.2 (Pin_2), R1.1
- no-connect marks 6 -> 1
Other:
- note added: "Programming connector: Use any USB/serial adapter. Enter bootloader by bridging BOOT to GND during power-on or reset."
- note added: "Status/diagnostic LED indicators"
- note removed: "Status/diagnostic indicator"
- moved on the sheet: C1, H1, H2, R2, R3, R4, R8, TP2
