File: hardware/pcb-rev2/noisemeter.kicad_pcb (KiCad board)
At the start: 2 copper layers, 44 x 37.8 mm, 23 parts, among them J1 USB_B_Micro, SW1 SW_Push, U1 AP2112K-3.3, U2 ESP32-C3-MINI-1-N4

Commit message: finalize rev2 design
Parts:
- moved C3 2.99 mm to (166.2, 98.2), turned to 90 degrees
Routing:
- net +3V3: track 49.4 -> 42.5 mm, vias 3 -> 5
- net GND: vias 23 -> 21
