File: hardware/pcb-rev2/noisemeter.kicad_sch (KiCad schematic)
At the start: 23 parts, among them J1 USB_B_Micro, SW1 SW_Push, U1 AP2112K-3.3, U2 ESP32-C3-MINI-1-N4

Commit message: finalize rev2 design
Parts:
- C1, C2, C3: NWI Part # (none) -> 000191-1-00-102-010123-00
- C4: NWI Part # (none) -> 000000-0-00-102-010012-00; Part Number CL21A106KOQNNNE -> CL21A106KPFNNNF
- C5, C6: NWI Part # (none) -> 000000-0-00-102-000061-00
- C7: Part Number CL10B201KB8NNNC -> CC0603KRX7R9BB201
- D1: NWI Part # (none) -> 000000-0-00-104-000114-00
- H1, H2, TP1: now left out of the parts list
- R10, R2, R3, R8: NWI Part # (none) -> 095004-4-00-101-011420-01
- R4, R5, R6: NWI Part # (none) -> 000000-0-00-101-010134-01
- U2: NWI Part # (none) -> 000000-0-00-106-000454-01
Changed lines of the file:
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@@
   (title_block
     (title "Noisemeter Device")
-    (date "2024-01-28")
+    (date "2024-02-07")
     (rev "2")
     (company "Civic Tech Toronto")
@@
     )
     (property "Part Number" "ESP32-C3-MINI-1-N4" (at 113.03 100.33 0)
+      (effects (font (size 1.27 1.27)) hide)
+    )
+    (property "NWI Part #" "000000-0-00-106-000454-01" (at 113.03 100.33 0)
       (effects (font (size 1.27 1.27)) hide)
     )
@@
       (effects (font (size 1.27 1.27)) hide)
     )
+    (property "NWI Part #" "000000-0-00-104-000114-00" (at 229.235 102.235 0)
+      (effects (font (size 1.27 1.27)) hide)
+    )
     (pin "1")
     (pin "2")
@@
   )
   (symbol (lib_id "Mechanical:MountingHole") (at 139.7 184.15 0) (unit 1)
-    (in_bom yes) (on_board yes) (dnp no) (fields_autoplaced)
+    (in_bom no) (on_board yes) (dnp no) (fields_autoplaced)
     (property "Reference" "H2" (at 142.24 181.61 0)
       (effects (font (size 1.27 1.27)) (justify left))
@@
     )
     (property "Datasheet" "~" (at 139.7 184.15 0)
+      (effects (font (size 1.27 1.27)) hide)
+    )
+    (property "NWI Part #" "" (at 139.7 184.15 0)
       (effects (font (size 1.27 1.27)) hide)
     )
@@
       (effects (font (size 1.27 1.27)) hide)
     )
+    (property "NWI Part #" "000000-0-00-101-010134-01" (at 111.76 149.225 0)
+      (effects (font (size 1.27 1.27)) hide)
+    )
     (pin "1")
     (pin "2")
@@
       (effects (font (size 1.27 1.27)) hide)
     )
+    (property "NWI Part #" "" (at 222.885 135.89 0)
+      (effects (font (size 1.27 1.27)) hide)
+    )
     (pin "1")
     (pin "2")
@@
     )
     (property "Part Number" "0473461001" (at 51.435 41.91 0)
+      (effects (font (size 1.27 1.27)) hide)
+    )
+    (property "NWI Part #" "" (at 51.435 41.91 0)
       (effects (font (size 1.27 1.27)) hide)
     )
@@
       (effects (font (size 1.27 1.27)) hide)
     )
+    (property "NWI Part #" "000000-0-00-102-000061-00" (at 155.575 87.63 0)
+      (effects (font (size 1.27 1.27)) hide)
+    )
     (pin "1")
     (pin "2")
@@
   )
   (symbol (lib_id "Connector:TestPoint") (at 130.81 97.79 270) (unit 1)
-    (in_bom yes) (on_board yes) (dnp no)
+    (in_bom no) (on_board yes) (dnp no)
     (property "Reference" "TP1" (at 135.89 97.79 90)
       (effects (font (size 1.27 1.27)) (justify left))
@@
     )
     (property "Datasheet" "~" (at 130.81 102.87 0)
+      (effects (font (size 1.27 1.27)) hide)
+    )
+    (property "NWI Part #" "" (at 130.81 97.79 0)
       (effects (font (size 1.27 1.27)) hide)
     )
@@
       (effects (font (size 1.27 1.27)) hide)
     )
+    (property "NWI Part #" "000191-1-00-102-010123-00" (at 91.44 40.64 0)
+      (effects (font (size 1.27 1.27)) hide)
+    )
     (pin "1")
     (pin "2")
@@
       (effects (font (size 1.27 1.27)) hide)
     )
+    (property "NWI Part #" "095004-4-00-101-011420-01" (at 215.265 102.235 0)
+      (effects (font (size 1.27 1.27)) hide)
+    )
     (pin "1")
     (pin "2")
@@
       (effects (font (size 1.27 1.27)) hide)
     )
+    (property "NWI Part #" "095004-4-00-101-011420-01" (at 68.58 102.87 0)
+      (effects (font (size 1.27 1.27)) hide)
+    )
     (pin "1")
     (pin "2")
@@
     )
     (property "Part Number" "CL10A105KA8NNNC" (at 115.57 40.64 0)
+      (effects (font (size 1.27 1.27)) hide)
+    )
+    (property "NWI Part #" "000191-1-00-102-010123-00" (at 115.57 40.64 0)
       (effects (font (size 1.27 1.27)) hide)
     )
@@
       (effects (font (size 1.27 1.27)) hide)
     )
+    (property "NWI Part #" "000000-0-00-101-010134-01" (at 111.76 152.4 0)
+      (effects (font (size 1.27 1.27)) hide)
+    )
     (pin "1")
     (pin "2")
@@
       (effects (font (size 1.27 1.27)) hide)
     )
+    (property "NWI Part #" "095004-4-00-101-011420-01" (at 68.58 105.41 0)
+      (effects (font (size 1.27 1.27)) hide)
+    )
     (pin "1")
     (pin "2")
@@
       (effects (font (size 1.27 1.27)) hide)
     )
+    (property "NWI Part #" "000000-0-00-101-010134-01" (at 74.93 83.82 0)
+      (effects (font (size 1.27 1.27)) hide)
+    )
     (pin "1")
     (pin "2")
@@
     )
     (property "Part Number" "AP2112K-3.3" (at 103.505 40.64 0)
+      (effects (font (size 1.27 1.27)) hide)
+    )
+    (property "NWI Part #" "" (at 103.505 40.64 0)
       (effects (font (size 1.27 1.27)) hide)
     )
@@
       (effects (font (size 1.27 1.27)) hide)
     )
+    (property "NWI Part #" "000000-0-00-102-000061-00" (at 244.475 40.64 0)
+      (effects (font (size 1.27 1.27)) hide)
+    )
     (pin "1")
     (pin "2")
@@
       (effects (font (size 1.27 1.27)) hide)
     )
-    (property "Part Number" "CL21A106KOQNNNE" (at 145.415 87.63 0)
+    (property "Part Number" "CL21A106KPFNNNF" (at 145.415 87.63 0)
+      (effects (font (size 1.27 1.27)) hide)
+    )
+    (property "NWI Part #" "000000-0-00-102-010012-00" (at 145.415 87.63 0)
       (effects (font (size 1.27 1.27)) hide)
     )
@@
     )
     (property "Part Number" "CL10A105KA8NNNC" (at 74.93 90.17 0)
+      (effects (font (size 1.27 1.27)) hide)
+    )
+    (property "NWI Part #" "000191-1-00-102-010123-00" (at 74.93 90.17 0)
       (effects (font (size 1.27 1.27)) hide)
     )
@@
     )
     (property "Part Number" "SPH0645LM4H-B" (at 219.075 55.88 0)
+      (effects (font (size 1.27 1.27)) hide)
+    )
+    (property "NWI Part #" "" (at 219.075 55.88 0)
       (effects (font (size 1.27 1.27)) hide)
     )
@@
       (effects (font (size 1.27 1.27)) hide)
     )
+    (property "NWI Part #" "095004-4-00-101-011420-01" (at 240.665 55.88 0)
+      (effects (font (size 1.27 1.27)) hide)
+    )
     (pin "1")
     (pin "2")
@@
       (effects (font (size 1.27 1.27)) hide)
     )
-    (property "Part Number" "CL10B201KB8NNNC" (at 253.365 40.64 0)
+    (property "Part Number" "CC0603KRX7R9BB201" (at 253.365 40.64 0)
+      (effects (font (size 1.27 1.27)) hide)
+    )
+    (property "NWI Part #" "" (at 253.365 40.64 0)
       (effects (font (size 1.27 1.27)) hide)
     )
@@
   )
   (symbol (lib_id "Mechanical:MountingHole") (at 139.7 177.8 0) (unit 1)
-    (in_bom yes) (on_board yes) (dnp no) (fields_autoplaced)
+    (in_bom no) (on_board yes) (dnp no) (fields_autoplaced)
     (property "Reference" "H1" (at 142.24 175.26 0)
       (effects (font (size 1.27 1.27)) (justify left))
@@
       (effects (font (size 1.27 1.27)) hide)
     )
+    (property "NWI Part #" "" (at 139.7 177.8 0)
+      (effects (font (size 1.27 1.27)) hide)
+    )

Commit message: final edits and bom changes
Parts:
- C1, C2, C3: Part Number CL10A105KA8NNNC -> CC0603KRX5R6BB105
- C4: Part Number CL21A106KPFNNNF -> CL21A106KPFNNNG
- C5, C6: Part Number CL10B104KA8NNNC -> CC0603KRX7R6BB104
- C7: Part Number CC0603KRX7R9BB201 -> 06033A201FAT2A
- D1: Part Number LTST-C190GKT -> APT1608LVBC/D
- J1: Part Number 0473461001 -> 0473460001
- U1: Part Number AP2112K-3.3 -> AP2112K-3.3TRG1
Changed lines of the file:
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@@
       (effects (font (size 1.27 1.27)) hide)
     )
-    (property "Part Number" "LTST-C190GKT" (at 229.235 102.235 0)
+    (property "Part Number" "APT1608LVBC/D" (at 229.235 102.235 0)
       (effects (font (size 1.27 1.27)) hide)
     )
@@
       (effects (font (size 1.27 1.27)) hide)
     )
-    (property "Part Number" "0473461001" (at 51.435 41.91 0)
+    (property "Part Number" "0473460001" (at 51.435 41.91 0)
       (effects (font (size 1.27 1.27)) hide)
     )
@@
       (effects (font (size 1.27 1.27)) hide)
     )
-    (property "Part Number" "CL10B104KA8NNNC" (at 155.575 87.63 0)
+    (property "Part Number" "CC0603KRX7R6BB104" (at 155.575 87.63 0)
       (effects (font (size 1.27 1.27)) hide)
     )
@@
       (effects (font (size 1.27 1.27)) hide)
     )
-    (property "Part Number" "CL10A105KA8NNNC" (at 91.44 40.64 0)
+    (property "Part Number" "CC0603KRX5R6BB105" (at 91.44 40.64 0)
       (effects (font (size 1.27 1.27)) hide)
     )
@@
       (effects (font (size 1.27 1.27)) hide)
     )
-    (property "Part Number" "CL10A105KA8NNNC" (at 115.57 40.64 0)
+    (property "Part Number" "CC0603KRX5R6BB105" (at 115.57 40.64 0)
       (effects (font (size 1.27 1.27)) hide)
     )
@@
       (effects (font (size 1.27 1.27)) hide)
     )
-    (property "Part Number" "AP2112K-3.3" (at 103.505 40.64 0)
+    (property "Part Number" "AP2112K-3.3TRG1" (at 103.505 40.64 0)
       (effects (font (size 1.27 1.27)) hide)
     )
@@
       (effects (font (size 1.27 1.27)) hide)
     )
-    (property "Part Number" "CL10B104KA8NNNC" (at 244.475 40.64 0)
+    (property "Part Number" "CC0603KRX7R6BB104" (at 244.475 40.64 0)
       (effects (font (size 1.27 1.27)) hide)
     )
@@
       (effects (font (size 1.27 1.27)) hide)
     )
-    (property "Part Number" "CL21A106KPFNNNF" (at 145.415 87.63 0)
+    (property "Part Number" "CL21A106KPFNNNG" (at 145.415 87.63 0)
       (effects (font (size 1.27 1.27)) hide)
     )
@@
       (effects (font (size 1.27 1.27)) hide)
     )
-    (property "Part Number" "CL10A105KA8NNNC" (at 74.93 90.17 0)
+    (property "Part Number" "CC0603KRX5R6BB105" (at 74.93 90.17 0)
       (effects (font (size 1.27 1.27)) hide)
     )
@@
       (effects (font (size 1.27 1.27)) hide)
     )
-    (property "Part Number" "CC0603KRX7R9BB201" (at 253.365 40.64 0)
-      (effects (font (size 1.27 1.27)) hide)
-    )
+    (property "Part Number" "06033A201FAT2A" (at 253.365 40.64 0)
+      (effects (font (size 1.27 1.27)) hide)
+    )
