File: hardware/pcb-rev3/noisemeter.kicad_pcb (KiCad board)
At the start: 2 copper layers, 44 x 31 mm, 19 parts, among them J1 USB_B_Micro, SW1 SW_Push, U1 AP2112K-3.3, U2 ESP32-C3-MINI-1-N4

Commit message: minor schematic fixes
Other:
- board text removed: ";.x_t} {\H0.62500x;(Part number and text placement/orientation on our products are }{\H0.62500x;subject to change,} {\H0.62500x;we do not recommend using them as a locating reference for }{\H0.62500x;modification purposes)}"
- board text removed: "A"
- board text removed: "B"
- board text removed: "END VIEW"
- board text removed: "INSIDE BOX"
- board text removed: "INSIDE LID"
- board text removed: "MAXIMUM"
- board text removed: "P.C. BOARD SIZE"
- board text removed: "SECTION A-A"
- board text removed: "SECTION B-B"
- board text removed: "SIDE VIEW"
- board text removed: "TOP VIEW"
- board text removed: "{\H2.0000;Dimensions:}\fArial|b0|i0;{\H2.0000; mm [inches]}"
- board text removed: "{\H2.0000;www.hammondmfg.com}"

Commit message: cleaning up layout
Parts:
- added D2: ESD5Z3.3T5G, Diode_SMD:D_0603_1608Metric, F.Cu at (167.5, 97.6)
- added U3: USBLC6-2SC6, Package_TO_SOT_SMD:SOT-23-6, F.Cu at (167.4, 88.5)
- C1, C2, C3: value 1U -> 1uF
- C4: value 10U -> 10uF
- C5, C6: value 0.1U -> 0.1uF
- C7: value 200P -> 200pF
- moved C2 1.93 mm to (149.8, 96.0)
- moved U1 1.93 mm to (146.8, 96.0)
- moved C3 1.79 mm to (143.8, 98.3), turned to -90 degrees
- moved C6 1.50 mm to (140.2, 95.5)
- moved C7 1.50 mm to (138.6, 95.5)
- moved R8 1.14 mm to (153.1, 88.7), turned to 180 degrees
- moved D1 0.70 mm to (167.5, 100.8)
- moved J1 0.65 mm to (171.9, 92.0)
- moved TP1 0.14 mm to (162.9, 88.9)
Connections:
- J1 pad 2: USB_D_N -> USB_in_D_N
- J1 pad 3: USB_D_P -> USB_in_D_P
Routing:
- net VBUS: track 3.62 -> 31.3 mm, vias 0 -> 2
- net +3V3: track 32.9 -> 49.4 mm
- net USB_D_N: track 11.8 -> 3.82 mm
- net USB_D_P: track 11.8 -> 5.43 mm
- net USB_in_D_N: track 0.00 -> 5.80 mm
- net FACT_RESET: track 34.4 -> 29.8 mm
- net USB_in_D_P: track 0.00 -> 4.25 mm
- net Net-(D1-K): track 26.1 -> 23.3 mm
- removed copper zone on B.Cu, net +3V3
- removed copper zone on F.Cu, net VBUS
