File: hardware/pcb-rev4/noisemeter.kicad_pcb (KiCad board)
At the start: 2 copper layers, 44 x 31 mm, 27 parts, among them J1 USB_B_Micro, SW1 SW_Push, U1 AP2112K-3.3, U2 USBLC6-2SC6, U3 ESP32-S3-MINI-1, U4 IM64A130A

Commit message: finalize rev4 hardware
Parts:
- added TP5: TestPoint, TestPoint:TestPoint_Pad_D1.0mm, F.Cu at (168.0, 86.8)
- added TP6: TestPoint, TestPoint:TestPoint_Pad_D1.0mm, F.Cu at (166.0, 86.8)
- added TP7: TestPoint, TestPoint:TestPoint_Pad_D1.0mm, F.Cu at (166.0, 84.8)
- U4: value IM64A130A -> IM64D130A
- moved TP2 2.83 mm to (168.0, 82.8)
- moved TP4 2.83 mm to (168.0, 84.8)
- moved R5 1.35 mm to (146.8, 82.8)
- moved R6 1.25 mm to (146.8, 81.2)
Connections:
- U3 pad 31: GND -> Net-(U3-IO35)
- U3 pad 32: GND -> Net-(U3-IO36)
- U3 pad 33: GND -> Net-(U3-IO37)
- U3 pad 41: GND -> unconnected-(U3-IO45-Pad41)
- U3 pad 44: GND -> unconnected-(U3-IO46-Pad44)
Routing:
- net Net-(U3-IO35): track 0.00 -> 5.83 mm
- net Net-(U3-IO37): track 0.00 -> 4.97 mm
- net Net-(U3-IO36): track 0.00 -> 4.06 mm
- net Net-(U3-TXD0): track 3.16 -> 5.02 mm
- net Net-(U3-IO0): track 3.44 -> 2.19 mm
- net Net-(U3-IO3): track 3.22 -> 2.09 mm
