File: hardware/pcb-rev4/noisemeter.kicad_sch (KiCad schematic)
At the start: 26 parts, among them J1 USB_B_Micro, SW1 SW_Push, U1 AP2112K-3.3, U2 USBLC6-2SC6, U3 ESP32-S3-MINI-1, U4 IM64A130A

Commit message: finalize rev4 hardware
Parts:
- added TP5, TP6, TP7: TestPoint, TestPoint:TestPoint_Pad_D1.0mm, symbol Connector:TestPoint
- U4: value IM64A130A -> IM64D130A
Connections:
- net GND: no longer U3.31 (IO35), U3.32 (IO36), U3.33 (IO37), U3.41 (IO45), U3.44 (IO46)
- new net: TP6.1, U3.32 (IO36)
- new net: TP5.1, U3.31 (IO35)
- new net: TP7.1, U3.33 (IO37)
- no-connect marks 2 -> 4
Other:
- note added: "Boot pins w/ internal pull-down"
